File: MCU Datalogger.kicad_sch (KiCad schematic)
At the start: 0 parts

Commit message: Have added required symbols to the schematic sheets.
Parts:
- added BT1: Battery, symbol Device:Battery
- added C1, C2, C3, C4: C, symbol Device:C
- added C5: C_Polarized, symbol Device:C_Polarized
- added D1, D2: LED, symbol Device:LED
- added H1, H2, H3, H4: MountingHole, symbol Mechanical:MountingHole
- added R1, R2, R3, R4, R5, R6, R7: R, symbol Device:R
- added U1, U2: 24LC1025, symbol Memory_EEPROM:24LC1025
- added U3: DS1337S_, DS1337S_:SOIC127P600X175-8N, symbol DS1337S_:DS1337S_
- added U4: ATMEGA328P-AU, ATMEGA328P-AU:QFP80P900X900X120-32N, symbol ATMEGA328P-AU:ATMEGA328P-AU
- added Y1, Y2: Crystal, symbol Device:Crystal
Connections:
- new net: U4.21 (GND), U4.3 (GND), U4.5 (GND)
- new net: U4.4 (VCC), U4.6 (VCC)
Other:
- added sheet Connectors (Connectors.kicad_sch)
- title: (none) -> ${project_name}
