File: MCU Datalogger.kicad_sch (KiCad schematic)
At the start: 25 parts, among them U1 24LC1025, U2 24LC1025, U3 DS1337S_, U4 ATMEGA328P-AU, Y1 16 MHz, Y2 32.768 KHz

Commit message: Add files via upload
Connections:
- net SCK: no longer R1.2, U1.6 (SCL), U2.6 (SCL), U3.6 (SCL), U4.28 (PC5)
- net Vcc: now also BT1.1 (+), C5.1, D1.2 (A), U4.18 (AVCC), U4.4 (VCC)
- new net SCL: R1.2, U1.6 (SCL), U2.6 (SCL), U3.6 (SCL), U4.28 (PC5)
Other:
- sheet Connectors ports: added SCL; removed none
Changed lines of the file:
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@@
 	(wire
 		(pts
-			(xy 137.16 137.16) (xy 139.7 137.16)
+			(xy 137.16 134.62) (xy 139.7 134.62)
 		)
 		(stroke
@@
 	(wire
 		(pts
-			(xy 236.22 43.18) (xy 236.22 48.26)
-		)
-		(stroke
-			(width 0)
-			(type default)
-		)
-	)
-	(wire
-		(pts
 			(xy 88.9 68.58) (xy 88.9 73.66)
 		)
@@
 	(wire
 		(pts
+			(xy 137.16 142.24) (xy 139.7 142.24)
+		)
+		(stroke
+			(width 0)
+			(type default)
+		)
+	)
+	(wire
+		(pts
 			(xy 55.88 114.3) (xy 68.58 114.3)
 		)
@@
 	(wire
 		(pts
-			(xy 137.16 139.7) (xy 139.7 139.7)
+			(xy 137.16 137.16) (xy 139.7 137.16)
 		)
 		(stroke
@@
 		)
 	)
-	(label "SCK"
+	(label "SCL"
 		(at 91.44 110.49 0)
 		(effects
@@
 		)
 	)
-	(label "SCK"
+	(label "SCL"
 		(at 50.8 104.14 0)
 		(effects
@@
 		)
 	)
-	(label "SCK"
+	(label "SCL"
 		(at 182.88 91.44 0)
 		(effects
@@
 	)
 	(label "TX"
-		(at 137.16 137.16 180)
+		(at 137.16 134.62 180)
 		(effects
 			(font
@@
 		)
 	)
+	(label "Vcc"
+		(at 256.54 48.26 0)
+		(effects
+			(font
+				(size 1.27 1.27)
+			)
+			(justify left bottom)
+		)
+	)
 	(label "D2"
 		(at 218.44 60.96 0)
@@
 	)
 	(label "SCK"
+		(at 137.16 142.24 180)
+		(effects
+			(font
+				(size 1.27 1.27)
+			)
+			(justify right bottom)
+		)
+	)
+	(label "SCL"
 		(at 137.16 132.08 180)
 		(effects
@@
 	)
 	(label "RX"
-		(at 137.16 139.7 180)
+		(at 137.16 137.16 180)
 		(effects
 			(font
@@
 		)
 	)
-	(label "SCK"
+	(label "SCL"
 		(at 78.74 104.14 0)
 		(effects
@@
 		)
 	)
-	(label "SCK"
+	(label "SCL"
 		(at 45.72 50.8 0)
 		(effects
@@
 		(polyline
 			(pts
-				(xy 127 35.56) (xy 274.32 35.56) (xy 274.32 111.76) (xy 127 111.76)
+				(xy 177.8 119.38) (xy 198.12 119.38) (xy 198.12 149.86) (xy 177.8 149.86)
 			)
 			(stroke
@@
 		(polyline
 			(pts
-				(xy 177.8 119.38) (xy 198.12 119.38) (xy 198.12 149.86) (xy 177.8 149.86)
+				(xy 22.86 35.56) (xy 121.92 35.56) (xy 121.92 81.28) (xy 22.86 81.28)
 			)
 			(stroke
@@
 		(polyline
 			(pts
-				(xy 22.86 35.56) (xy 121.92 35.56) (xy 121.92 81.28) (xy 22.86 81.28)
+				(xy 127 35.56) (xy 274.32 35.56) (xy 274.32 111.76) (xy 127 111.76)
 			)
 			(stroke
@@
 	)
 	(symbol
-		(lib_id "power:PWR_FLAG")
-		(at 236.22 43.18 0)
-		(unit 1)
-		(exclude_from_sim no)
-		(in_bom yes)
-		(on_board yes)
-		(dnp no)
-		(fields_autoplaced yes)
-		(property "Reference" "#FLG01"
-			(at 236.22 41.275 0)
-			(effects
-				(font
-					(size 1.27 1.27)
-				)
-				(hide yes)
-			)
-		)
-		(property "Value" "PWR_FLAG"
-			(at 236.22 38.1 0)
-			(effects
-				(font
-					(size 1.27 1.27)
-				)
-			)
-		)
-		(property "Footprint" ""
-			(at 236.22 43.18 0)
-			(effects
-				(font
-					(size 1.27 1.27)
-				)
-				(hide yes)
-			)
-		)
-		(property "Datasheet" "~"
-			(at 236.22 43.18 0)
-			(effects
-				(font
-					(size 1.27 1.27)
-				)
-				(hide yes)
-			)
-		)
-		(property "Description" "Special symbol for telling ERC where power comes from"
-			(at 236.22 43.18 0)
-			(effects
-				(font
-					(size 1.27 1.27)
-				)
-				(hide yes)
-			)
-		)
-		(pin "1"
-		)
-		(instances
-			(project ""
-				(path "/19a27ba3-b273-42f4-b520-5672b9fc4c35"
-					(reference "#FLG01")
-					(unit 1)
-				)
-			)
-		)
-	)
-	(symbol
 		(lib_id "Device:R")
 		(at 91.44 104.14 0)
@@
 			)
 		)
-		(pin "SCK" passive
-			(at 139.7 132.08 180)
-			(effects
-				(font
-					(size 1.27 1.27)
-				)
-				(justify left)
-			)
-		)
 		(pin "TX" output
-			(at 139.7 137.16 180)
+			(at 139.7 134.62 180)
 			(effects
 				(font
@@
 		)
 		(pin "RX" input
-			(at 139.7 139.7 180)
+			(at 139.7 137.16 180)
 			(effects
 				(font
@@
 			(effects
 				(font
+					(size 1.27 1.27)
+				)
+				(justify left)
+			)
+		)
+		(pin "SCK" passive
+			(at 139.7 142.24 180)
+			(effects
+				(font
+					(size 1.27 1.27)
+				)
+				(justify left)
+			)
+		)
+		(pin "SCL" passive
+			(at 139.7 132.08 180)
+			(effects
+				(font
